File: 001_Simulation_und_Schaltungsentwurf/Schaltungsentwurf_v1/Schaltungsentwurf_v1/Schaltungsentwurf_v1.kicad_sch (KiCad schematic)
At the start: 57 parts, among them IC1 MPY634KP, IC2 MPY634KP, IC3 MPY634KP, J1 Screw_Terminal_01x04, U1 TL082, U2 TL082, U3 TL082

Commit message: Überarbeitung von SP und Plots
Parts:
- added TP10: V_in, TestPoint:TestPoint_Loop_D1.80mm_Drill1.0mm_Beaded, symbol 000_My_Symbols:Testpoint
Connections:
- net V_in: now also TP10.1
- net Vc_DC: no longer names the net of JP5.2 (C), R11.2, TP4.1
Other:
- moved on the sheet: C1, C2, C3, C4, C5, C6, H1, H2, H3, H4, IC1, IC2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
