File: 001_Simulation_und_Schaltungsentwurf/005_selfe_tuned_filter/selfe_tuned_filter.kicad_sch (KiCad schematic)
At the start: 37 parts, among them IC1 MPY634KP, IC2 MPY634KP, IC3 MPY634KP, J1 Screw_Terminal_01x04, U1 TL082, U2 TL082, U3 TL082

Commit message: Stand 24.10
Parts:
- removed C1, C2, C3: 100n, Capacitor_THT:C_Disc_D3.0mm_W2.0mm_P2.50mm, symbol Device:C
- removed H1, H2, H3, H4: MountingHole, MountingHole:MountingHole_2.2mm_M2_DIN965, symbol Mechanical:MountingHole
- removed J1: Screw_Terminal_01x04, TerminalBlock:TerminalBlock_Altech_AK300-4_P5.00mm, symbol Connector:Screw_Terminal_01x04
- removed TP1: BPF, TestPoint:TestPoint_Loop_D1.80mm_Drill1.0mm_Beaded, symbol 000_My_Symbols:Testpoint
- removed TP2: LPF, TestPoint:TestPoint_Loop_D1.80mm_Drill1.0mm_Beaded, symbol 000_My_Symbols:Testpoint
- removed TP3: HPF, TestPoint:TestPoint_Loop_D1.80mm_Drill1.0mm_Beaded, symbol 000_My_Symbols:Testpoint
- removed TP4: BSF, TestPoint:TestPoint_Loop_D1.80mm_Drill1.0mm_Beaded, symbol 000_My_Symbols:Testpoint
- removed TP5: V_in, TestPoint:TestPoint_Loop_D1.80mm_Drill1.0mm_Beaded, symbol 000_My_Symbols:Testpoint
- removed TP6: GND, TestPoint:TestPoint_Loop_D1.80mm_Drill1.0mm_Beaded, symbol 000_My_Symbols:Testpoint
- removed V3: 1, symbol Simulation_SPICE:VDC
- added V10: 10, symbol Simulation_SPICE:VDC
- added V8, V9: 15, symbol Simulation_SPICE:VDC
- V1: value 15 -> 1
- V2: value 15 -> 15.75
Connections:
- net +10V: now also V10.1; no longer IC1.14 (+VS), IC2.14 (+VS), IC3.14 (+VS), R7.2, U1.8 (V+), U2.8 (V+), U3.8 (V+), V1.1
- net GND: now also V2.2, V10.2, V8.1, V9.2; no longer V2.1
- net V_in: now also V1.1
- net -10V renamed -15V
- net -15V: now also V8.2; no longer V2.2
- net V_F3 renamed V_C
- new net: R7.2, V2.1
- new net +15V: IC1.14 (+VS), IC2.14 (+VS), IC3.14 (+VS), U1.8 (V+), U2.8 (V+), U3.8 (V+), V9.1
Other:
- note removed: ".param Rx = 10k Größe hängt davon ab, welche Eckfrequenz (Loop-Bandbreite / Gleichanteils­auskopplung) du haben willst und wie stark du den Ausgang belasten möchtest."
- note removed: "I/O"
- note removed: "Mounting Holes"
- note removed: "Supply Voltage"
- moved on the sheet: C4, C5, C6, IC1, IC2, IC3, R1, R10, R11, R12, R3, R4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

Commit message: Stand 04.11
Parts:
- R6: value {RCOM} -> 250
- R7: value {RCOM} -> 750
- V2: value 15.75 -> 14.2
Changed lines of the file:
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@@
 			)
 		)
-		(property "Value" "15.75"
+		(property "Value" "14.2"
 			(at 374.65 128.1401 0)
 			(effects
@@
 			)
 		)
-		(property "Value" "{RCOM}"
+		(property "Value" "250"
 			(at 364.49 110.49 90)
 			(effects
@@
 			)
 		)
-		(property "Value" "{RCOM}"
+		(property "Value" "750"
 			(at 373.38 119.3799 0)
 			(effects

Commit message: Lokale Änderungen am KiCad-Projekt gesichert
Parts:
- C5: value {CCOM} -> 1u
- R1: value {RCOM/H0} -> {1k/H0}
- R11, R4, R8, R9: value {RCOM} -> 1k
- R12: value {RCOM*Q} -> {1k*Q}
- R5: value {RCOM} -> {1k}
- R6: value 250 -> 1k
- R7: value 750 -> 1k
- V2: value 14.2 -> 2
Changed lines of the file:
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@@
 	(text_box "Integrator\nnew LP"
 		(exclude_from_sim yes)
-		(at 312.42 88.9 0)
-		(size 72.39 53.34)
+		(at 326.39 88.9 0)
+		(size 58.42 53.34)
 		(margins 0.9525 0.9525 0.9525 0.9525)
 		(stroke
@@
 			)
 		)
-		(property "Value" "{RCOM}"
+		(property "Value" "1k"
 			(at 181.61 100.33 90)
 			(effects
@@
 			)
 		)
-		(property "Value" "14.2"
+		(property "Value" "2"
 			(at 374.65 128.1401 0)
 			(effects
@@
 			)
 		)
-		(property "Value" "{RCOM}"
+		(property "Value" "1k"
 			(at 332.74 107.95 90)
 			(effects
@@
 			)
 		)
-		(property "Value" "{RCOM*Q}"
+		(property "Value" "{1k*Q}"
 			(at 116.84 140.97 90)
 			(effects
@@
 			)
 		)
-		(property "Value" "250"
+		(property "Value" "1k"
 			(at 364.49 110.49 90)
 			(effects
@@
 			)
 		)
-		(property "Value" "{RCOM/H0}"
+		(property "Value" "{1k/H0}"
 			(at 116.84 148.59 90)
 			(effects
@@
 			)
 		)
-		(property "Value" "{CCOM}"
+		(property "Value" "1u"
 			(at 349.2563 96.52 90)
 			(effects
@@
 			)
 		)
-		(property "Value" "{RCOM}"
+		(property "Value" "{1k}"
 			(at 140.97 130.81 90)
 			(effects
@@
 			)
 		)
-		(property "Value" "{RCOM}"
+		(property "Value" "1k"
 			(at 205.74 90.17 90)
 			(effects
@@
 			)
 		)
-		(property "Value" "{RCOM}"
+		(property "Value" "1k"
 			(at 181.61 107.95 90)
 			(effects
@@
 			)
 		)
-		(property "Value" "750"
+		(property "Value" "1k"
 			(at 373.38 119.3799 0)
 			(effects

Commit message: Stand 14.11
Parts:
- removed IC3: MPY634KP, symbol BA_Footprints:MPY634KP
- added IC4: MPY634KP, symbol BA_Footprints:MPY634KP
- added V3: 0.1, symbol Simulation_SPICE:VDC
- R5: value {1k} -> 1k
Connections:
- net +10V: now also IC4.4 (SCALE_FACTOR)
- net +15V: now also IC4.14 (+VS)
- net -15V: now also IC4.8 (-VS)
- net GND: now also IC4.10 (Z_2_INPUT), IC4.2 (X_2_INPUT), IC4.7 (Y_2_INPUT), V3.2
- net HPF: now also V3.1
- net LPF: now also IC4.1 (X_1_INPUT)
- net V_C: now also IC4.6 (Y_1_INPUT)
- net mult3_out: now also IC4.11 (Z_1_INPUT), IC4.12 (OUTPUT)
Other:
- note added: ".control op print all .endc"
- note added: ".param RCOM = 1k .param CCOM = 1u .param Q = 0.707 .param H0 = 1"
- note removed: ".control set controlswait write selfe_tuned_filter.raw all .endc"
- note removed: ".param RCOM = 1k .param CCOM = 1u .param Q = 1 .param H0 = 1"
- moved on the sheet: C4, C5, C6, IC1, IC2, R1, R10, R11, R12, R3, R4, R5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
