File: 001_Simulation_und_Schaltungsentwurf/006_Schaltungsentwurf_v1/Schaltungsentwurf_v1.kicad_sch (KiCad schematic)
At the start: 69 parts, among them IC1 MPY634KP, IC2 MPY634KP, IC3 MPY634KP, J1 Screw_Terminal_01x04, U1 TL082, U2 TL082, U3 MCP4261-104E_P, U4 MCP4261-104E_P, U5 TL082

Commit message: Lokale Änderungen am KiCad-Projekt gesichert
Parts:
- removed JP2: SF1, 000_OUF:Connector 2 Pin 2.54mm, symbol Jumper:Jumper_2_Open
- removed JP3: SF2, 000_OUF:Connector 2 Pin 2.54mm, symbol Jumper:Jumper_2_Open
- removed JP4: SF3, 000_OUF:Connector 2 Pin 2.54mm, symbol Jumper:Jumper_2_Open
- added C11, C12, C13: 100n, 000_OUF:100nF, symbol Device:C_Small
- added JP2, JP3, JP4: ~, 000_OUF:Connector 2 Pin 2.54mm, symbol Jumper:Jumper_2_Small_Open
- added TP14: ZCD, 000_OUF:TestPoint, symbol 000_My_Symbols:Testpoint
- added TP15: FFT, 000_OUF:TestPoint, symbol 000_My_Symbols:Testpoint
- TP6: value SHDN1 -> SHDN2
Connections:
- net +15V: now also C11.1, C12.1, C13.1
- net -15V: now also C11.2, C12.2, C13.2
- net FFT: now also TP15.1
- net ZCD: now also TP14.1
- net at IC3.4 (SCALE_FACTOR): now also JP4.2 (B)
- net at RV1.1, RV1.2: now also JP2.1 (A)
- net at IC1.4 (SCALE_FACTOR): now also JP2.2 (B)
- net at RV3.1, RV3.2: now also JP4.1 (A)
- net at IC2.4 (SCALE_FACTOR): now also JP3.2 (B)
- net at RV2.1, RV2.2: now also JP3.1 (A)

Commit message: Stand 14.11
Parts:
- C1, C3, C5: value {CCOM} -> 1u
- R2, R3, R4, R5, R9: value {RCOM} -> 1k
- RV1, RV2, RV4, RV5, RV6: footprint 000_OUF:Trimmer Rund -> Potentiometer_THT:Potentiometer_Bourns_3296Y_Vertical
- RV3: footprint 000_OUF:Trimmer straight -> Potentiometer_THT:Potentiometer_Bourns_3296Y_Vertical
Connections:
- net -10V is gone; now on net -15V: RV1.3, RV2.3, RV3.3
- no-connect marks 12 -> 16

Commit message: Erste Iteration des PCBs
Parts:
- removed PS1: LM2576WT, Package_TO_SOT_THT:TO-220-5_Vertical, symbol AquaLift_lib:LM2576WT
- removed RV6: 5k, Potentiometer_THT:Potentiometer_Bourns_3296Y_Vertical, symbol Device:R_Potentiometer
- added J2, J3, J4, J5, J6: Conn_Coaxial, 001_CNC:BNC Edge Mount, symbol Connector:Conn_Coaxial
- added JP13: ~, 000_OUF:Connector 2 Pin 2.54mm, symbol Jumper:Jumper_2_Small_Open
- added TP16: mult1_out, 000_OUF:TestPoint, symbol 000_My_Symbols:Testpoint
- added TP17: mult2_out, 000_OUF:TestPoint, symbol 000_My_Symbols:Testpoint
- added TP18: mult3_out, 000_OUF:TestPoint, symbol 000_My_Symbols:Testpoint
- added U6: LM2596T-3.3, Package_TO_SOT_THT:TO-220-5_P3.4x3.7mm_StaggerOdd_Lead3.8mm_Vertical, symbol Regulator_Switching:LM2596T-3.3
- C7: value 100uF -> 470uF; footprint Capacitor_THT:C_Radial_D8.0mm_H11.5mm_P3.50mm -> Capacitor_THT:C_Radial_D10.0mm_H16.0mm_P5.00mm
- C9: value 1000uF -> 330uF
- D1: value MBR360 -> 1N5820; footprint 000_OUF:1N4001 -> Diode_THT:D_DO-27_P15.24mm_Horizontal
- JP1: value ~ -> R1_in
- JP10: value ~ -> RQ_out
- JP11: value ~ -> RH0_out
- JP5: value ~ -> R1_out
- JP6: value ~ -> R2_in
- JP7: value ~ -> RQ_in
- JP8: value ~ -> RH0_in
- JP9: value ~ -> R2_out
- L1: value 100uH -> 68uH; footprint Inductor_THT:L_Radial_D8.7mm_P5.00mm_Fastron_07HCP -> Inductor_THT:L_Radial_D12.0mm_P5.00mm_Fastron_11P
- R10, R11: value {RCOM} -> 1k
Connections:
- net +15V: now also U6.1 (VIN)
- net +3.3V: now also JP13.2 (B); no longer C9.1, L1.2
- net BPF: now also J4.1 (In)
- net BSF: now also J5.1 (In)
- net GND: now also J2.2 (Ext), J3.2 (Ext), J4.2 (Ext), J5.2 (Ext), J6.2 (Ext), U6.3 (GND), U6.5 (~{ON}/OFF)
- net HPF: now also J2.1 (In)
- net LPF: now also J3.1 (In)
- net V_in: now also J6.1 (In)
- net mult1_out: now also TP16.1
- net mult2_out: now also TP17.1
- net mult3_out: now also TP18.1
- net at D1.1 (K), L1.1: now also U6.2 (OUT)
- new net: C9.1, JP13.1 (A), L1.2, U6.4 (FB)
Other:
- moved on the sheet: C11, C12, C13, C2, C4, C7, C9, D1, IC1, IC2, IC3, JP2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

Commit message: documentation of the PCB (iteration 1)
Connections:
- net +3.3V: now also A1.39 (VSYS); no longer A1.36 (3V3)
Other:
- note removed: "V_out = 1.23V * (1 + (R_up/R_down))"
Changed lines of the file:
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@@
 		)
 	)
-	(text "V_out = 1.23V * (1 + (R_up/R_down))"
-		(exclude_from_sim no)
-		(at 375.412 244.094 0)
-		(effects
-			(font
-				(size 1.27 1.27)
-			)
-		)
-	)
 	(text_box "Poti 2\n\n"
 		(exclude_from_sim no)
@@
 	(wire
 		(pts
-			(xy 193.04 135.89) (xy 193.04 138.43)
+			(xy 182.88 135.89) (xy 182.88 138.43)
 		)
 		(stroke
@@
 	(symbol
 		(lib_id "power:+15V")
-		(at 193.04 135.89 0)
+		(at 182.88 135.89 0)
 		(unit 1)
 		(exclude_from_sim no)
@@
 		(dnp no)
 		(property "Reference" "#PWR022"
-			(at 193.04 139.7 0)
+			(at 182.88 139.7 0)
 			(effects
 				(font
@@
 		)
 		(property "Value" "+3.3V"
-			(at 194.31 134.62 0)
+			(at 184.15 134.62 0)
 			(effects
 				(font
@@
 		)
 		(property "Footprint" ""
-			(at 193.04 135.89 0)
+			(at 182.88 135.89 0)
 			(effects
 				(font
@@
 		)
 		(property "Datasheet" ""
-			(at 193.04 135.89 0)
+			(at 182.88 135.89 0)
 			(effects
 				(font
@@
 		)
 		(property "Description" "Power symbol creates a global label with name \"+15V\""
-			(at 193.04 135.89 0)
+			(at 182.88 135.89 0)
 			(effects
 				(font
